File: matrix.kicad_pcb (KiCad board)
At the start: 2 copper layers, 47 x 26.4 mm, 36 parts, among them U2 IS31FL3218-GR

Commit message: add name label, shuffle traces
Parts:
- R1: moved to F.Cu
- moved R1 7.95 mm to (58.8, 40.0)
Connections:
- A1 pad 19: /TOUCH_COMMON_SND -> /TOUCH_RCV_COL1
- A1 pad 20: /TOUCH_COMMON_SND -> /TOUCH_RCV_COL1
- A1 pad 22: /TOUCH_COMMON_SND -> /TOUCH_RCV_COL1
- A1 pad 25: /TOUCH_COMMON_SND -> /TOUCH_RCV_COL1
- CT11 pad 1: /TOUCH_COMMON_SND -> /TOUCH_RCV_COL1
- CT11 pad 2: /TOUCH_COMMON_SND -> /TOUCH_RCV_COL1
- CT12 pad 1: /TOUCH_COMMON_SND -> /TOUCH_RCV_COL1
- CT12 pad 2: /TOUCH_COMMON_SND -> /TOUCH_RCV_COL1
- CT13 pad 1: /TOUCH_COMMON_SND -> /TOUCH_RCV_COL1
- CT13 pad 2: (no net) -> /TOUCH_RCV_COL1
- CT14 pad 1: /TOUCH_COMMON_SND -> /TOUCH_RCV_COL1
- CT14 pad 2: (no net) -> /TOUCH_RCV_COL1
- CT21 pad 1: /TOUCH_COMMON_SND -> /TOUCH_RCV_COL1
- CT21 pad 2: /TOUCH_COMMON_SND -> /TOUCH_RCV_COL1
- CT22 pad 1: /TOUCH_COMMON_SND -> /TOUCH_RCV_COL1
- CT22 pad 2: /TOUCH_COMMON_SND -> /TOUCH_RCV_COL1
- CT23 pad 1: /TOUCH_COMMON_SND -> /TOUCH_RCV_COL1
- CT23 pad 2: (no net) -> /TOUCH_RCV_COL1
- CT24 pad 1: /TOUCH_COMMON_SND -> /TOUCH_RCV_COL1
- CT24 pad 2: (no net) -> /TOUCH_RCV_COL1
- CT31 pad 1: Net-(CT31-Pad1) -> /TOUCH_RCV_COL1
- CT31 pad 2: /TOUCH_COMMON_SND -> /TOUCH_RCV_COL1
- CT32 pad 1: Net-(CT31-Pad1) -> /TOUCH_RCV_COL1
- CT32 pad 2: /TOUCH_COMMON_SND -> /TOUCH_RCV_COL1
- CT41 pad 1: Net-(CT41-Pad1) -> /TOUCH_RCV_COL1
- CT41 pad 2: /TOUCH_COMMON_SND -> /TOUCH_RCV_COL1
- CT42 pad 1: Net-(CT41-Pad1) -> /TOUCH_RCV_COL1
- CT42 pad 2: /TOUCH_COMMON_SND -> /TOUCH_RCV_COL1
- D10 pad 3: (no net) -> /TOUCH_RCV_COL1
- D11 pad 3: (no net) -> /TOUCH_RCV_COL1
- D12 pad 3: (no net) -> /TOUCH_RCV_COL1
- D13 pad 3: (no net) -> /TOUCH_RCV_COL1
- D15 pad 3: (no net) -> /TOUCH_RCV_COL1
- D16 pad 3: (no net) -> /TOUCH_RCV_COL1
- D17 pad 3: (no net) -> /TOUCH_RCV_COL1
- D18 pad 3: (no net) -> /TOUCH_RCV_COL1
- D2 pad 3: (no net) -> /TOUCH_RCV_COL1
- D3 pad 3: (no net) -> /TOUCH_RCV_COL1
- D8 pad 3: (no net) -> /TOUCH_RCV_COL1
- D9 pad 3: (no net) -> /TOUCH_RCV_COL1
- R1 pad 1: /TOUCH_COMMON_SND -> /TOUCH_RCV_COL1
Routing:
- net /TOUCH_COMMON_SND: track 224.7 -> 0.00 mm, vias 8 -> 0
- net /TOUCH_RCV_COL1: track 0.00 -> 216.4 mm, vias 0 -> 9
- net Net-(A1-Pad26): track 1.98 -> 8.81 mm, vias 0 -> 1
- net /LP18: track 16.4 -> 17.1 mm
- net VCC: track 178.6 -> 177.9 mm
Other:
- board text added: "revision 1"
- board text added: "Матричка"

Commit message: cleanup
Parts:
- moved R1 0.63 mm to (58.8, 40.6)
Routing:
- net GND: track 86.9 -> 82.9 mm
- net /TOUCH_RCV_COL1: track 216.4 -> 213.7 mm
- net VCC: track 177.9 -> 175.7 mm
- net /LP21: track 30.6 -> 32.2 mm
Other:
- board size 47 x 26.4 mm -> 47.1 x 26.4 mm
- board text added: "touchy touch!"

Commit message: ready for production
Parts:
- R1, R3: footprint Resistor_SMD:R_0805_2012Metric -> Connector_PinHeader_2.54mm:PinHeader_1x02_P2.54mm_Vertical
- moved R3 6.85 mm to (25.4, 41.9)
- moved R1 2.30 mm to (61.0, 41.3), turned to 270 degrees
Connections:
- CT13 pad 2: /TOUCH_RCV_COL1 -> (no net)
- CT14 pad 2: /TOUCH_RCV_COL1 -> (no net)
- CT23 pad 2: /TOUCH_RCV_COL1 -> (no net)
- CT24 pad 2: /TOUCH_RCV_COL1 -> (no net)
- CT31 pad 1: /TOUCH_RCV_COL1 -> Net-(CT31-Pad1)
- CT32 pad 1: /TOUCH_RCV_COL1 -> Net-(CT31-Pad1)
- CT41 pad 1: /TOUCH_RCV_COL1 -> Net-(CT41-Pad1)
- CT42 pad 1: /TOUCH_RCV_COL1 -> Net-(CT41-Pad1)
- D10 pad 3: /TOUCH_RCV_COL1 -> (no net)
- D11 pad 3: /TOUCH_RCV_COL1 -> (no net)
- D12 pad 3: /TOUCH_RCV_COL1 -> (no net)
- D13 pad 3: /TOUCH_RCV_COL1 -> (no net)
- D15 pad 3: /TOUCH_RCV_COL1 -> (no net)
- D16 pad 3: /TOUCH_RCV_COL1 -> (no net)
- D17 pad 3: /TOUCH_RCV_COL1 -> (no net)
- D18 pad 3: /TOUCH_RCV_COL1 -> (no net)
- D2 pad 3: /TOUCH_RCV_COL1 -> (no net)
- D3 pad 3: /TOUCH_RCV_COL1 -> (no net)
- D8 pad 3: /TOUCH_RCV_COL1 -> (no net)
- D9 pad 3: /TOUCH_RCV_COL1 -> (no net)
Routing:
- net VCC: track 175.7 -> 171.6 mm
- net Net-(R3-Pad1): track 2.51 -> 6.46 mm
- net /TOUCH_RCV_COL1: track 213.7 -> 211.6 mm, vias 9 -> 8
- net Net-(A1-Pad26): track 8.67 -> 9.95 mm, vias 1 -> 0
- net GND: track 82.9 -> 81.9 mm
